File: nrf52840_dev.kicad_sch (KiCad schematic)
At the start: 19 parts, among them J1 SWD, J10 POWER, J2 SPI1, J3 POWER, J4 Conn_01x01, J5 Conn_01x01, J6 SPI2, J7 POWER, J8 Conn_01x01, J9 Conn_01x01

Commit message: Small fix
Parts:
- removed DC1: DC-DC, mini360:DC-DC mini360, symbol dc-dc:DC-DC
- removed H1: MountingHole, MountingHole:MountingHole_3.2mm_M3, symbol Mechanical:MountingHole
- removed J1: SWD, Connector_PinHeader_2.54mm:PinHeader_1x03_P2.54mm_Vertical, symbol Connector_Generic:Conn_01x03
- removed J10, J3, J7: POWER, Connector_PinHeader_2.54mm:PinHeader_1x02_P2.54mm_Vertical, symbol Connector_Generic:Conn_01x02
- removed J2: SPI1, Connector_PinHeader_2.54mm:PinHeader_1x03_P2.54mm_Vertical, symbol Connector_Generic:Conn_01x03
- removed J4, J5, J8, J9: Conn_01x01, Connector_PinHeader_2.54mm:PinHeader_1x01_P2.54mm_Vertical, symbol Connector_Generic:Conn_01x01
- removed J6: SPI2, Connector_PinHeader_2.54mm:PinHeader_1x02_P2.54mm_Vertical, symbol Connector_Generic:Conn_01x02
- added C3, C4: C_Small, Capacitor_SMD:C_0603_1608Metric, symbol Device:C_Small
- added C32: 1F, Capacitor_THT:CP_Radial_D8.0mm_P3.50mm, symbol Device:CP1_Small
- added C5, C6: 0.1uF, Capacitor_SMD:C_0805_2012Metric, symbol Device:C_Small
- added D1: 1N4148, Diode_SMD:D_SOD-323, symbol Diode:1N4148
- added D3: NUP2105L, Package_TO_SOT_SMD:SOT-23, symbol Power_Protection:NUP2105L
- added H1, H2: MountingHole_Pad, MountingHole:MountingHole_3.2mm_M3_Pad_Via, symbol Mechanical:MountingHole_Pad
- added J1: Conn_01x04, Connector_JST:JST_XH_S4B-XH-A-1_1x04_P2.50mm_Horizontal, symbol Connector_Generic:Conn_01x04
- added J2: SWD, Connector_PinHeader_1.27mm:PinHeader_2x05_P1.27mm_Vertical_SMD, symbol Connector_Generic:Conn_02x05_Odd_Even
- added J4: Conn_Coaxial_Power, Connector_Coaxial:SMA_Amphenol_901-144_Vertical, symbol Connector:Conn_Coaxial_Power
- added JP1: terminator, Jumper:SolderJumper-2_P1.3mm_Open_RoundedPad1.0x1.5mm, symbol Jumper:SolderJumper_2_Open
- added R19: 100, Resistor_SMD:R_0805_2012Metric, symbol Device:R_Small
- added R6: 120, Resistor_SMD:R_0603_1608Metric, symbol Device:R_Small
- added U2: MCP2515-xSO, Package_SO:SOIC-18W_7.5x11.6mm_P1.27mm, symbol Interface_CAN_LIN:MCP2515-xSO
- added U5: SN65HVD230, Package_SO:SOIC-8_3.9x4.9mm_P1.27mm, symbol Interface_CAN_LIN:SN65HVD230
- added Y1: 8Mhz, Crystal:Crystal_HC49-U_Vertical, symbol Device:Crystal_Small
- D1, D2: footprint LED_THT:LED_D5.0mm -> LED_SMD:LED_1206_3216Metric
Connections:
- net 12VIN: now also J1.3 (Pin_3)
- net 3V3: now also C5.1, C6.1, J2.3 (Pin_3), R19.1, U2.18 (VDD), U5.3 (VCC)
- net CS: now also U1.12 (P0.26), U2.16 (~{CS}); no longer U1.33 (P0.13)
- net GND: now also C3.2, C32.2, C4.2, C5.2, C6.2, D3.3 (A), H1.1, H2.1, J1.4 (Pin_4), J2.6 (Pin_6), J2.9 (Pin_9), J4.2 (Ext), U2.9 (VSS), U5.2 (GND), U5.8 (Rs)
- net IRQ: now also U1.17 (P1.09), U2.12 (~{INT}); no longer U1.35 (P0.24)
- net MISO: now also U2.15 (SO)
- net MOSI: now also U2.14 (SI)
- net RX: now also U1.22 (P0.07); no longer U1.12 (P0.26)
- net SCK: now also U2.13 (SCK)
- net SWD_CLK: now also J2.7 (Pin_7)
- net SWD_IO: now also J2.5 (Pin_5)
- net MCP_RST: now reaches U1.10 (P0.30(AIN6))
- net MCP_RST: now also U2.17 (~{RESET})
- new net: D1.2 (A), R19.2
- new net: C3.1, U2.8 (OSC1), Y1.1
- new net: C4.1, U2.7 (OSC2), Y1.2
- new net: U2.1 (TXCAN), U5.1 (D)
- new net: U2.2 (RXCAN), U5.4 (R)
- new net: JP1.1 (A), R6.2
- new net 5V: J2.1 (Pin_1)
- new net CANH: D3.1 (K), J1.1 (Pin_1), R6.1, U5.7 (CANH)
- new net CANL: D3.2 (K), J1.2 (Pin_2), JP1.2 (B), U5.6 (CANL)
- new net ublox/GPS_RF: J4.1 (In)
- new net ublox/GPS_VBAT: C32.1, D1.1 (K)
- no-connect marks 0 -> 36
Other:
- added sheet power (s1st14.kicad_sch)
- added sheet ublox (ubloxM8N.kicad_sch)
- note added: "CAN BUS"
- note added: "GPS"
- note added: "MCU"
- moved on the sheet: C1, C2, D1, D2, R1, R2, U1

Commit message: fixes
Parts:
- added LOGO1: ~, logo:logo_15x9, symbol logo:logo15x9
- H1, H2, JP1: now left out of the parts list
- Y1: footprint Crystal:Crystal_HC49-U_Vertical -> Crystal:Crystal_HC49-4H_Vertical
Changed lines of the file:
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@@
       (effects (font (size 1.27 1.27)) (justify right))
     )
-    (property "Footprint" "Crystal:Crystal_HC49-U_Vertical" (at 151.765 62.23 0)
+    (property "Footprint" "Crystal:Crystal_HC49-4H_Vertical" (at 151.765 62.23 0)
       (effects (font (size 1.27 1.27)) hide)
     )
@@
   )
   (symbol (lib_id "Mechanical:MountingHole_Pad") (at 131.445 186.055 0) (unit 1)
-    (in_bom yes) (on_board yes) (dnp no) (fields_autoplaced)
+    (in_bom no) (on_board yes) (dnp no) (fields_autoplaced)
     (property "Reference" "H2" (at 134.62 183.515 0)
       (effects (font (size 1.27 1.27)) (justify left))
@@
   )
   (symbol (lib_id "Jumper:SolderJumper_2_Open") (at 257.175 35.56 0) (unit 1)
-    (in_bom yes) (on_board yes) (dnp no)
+    (in_bom no) (on_board yes) (dnp no)
     (property "Reference" "JP1" (at 262.89 31.75 0)
       (effects (font (size 1.27 1.27)))
@@
     )
   )
+  (symbol (lib_id "logo:logo15x9") (at 158.75 175.26 0) (unit 1)
+    (in_bom no) (on_board yes) (dnp no)
+    (property "Reference" "LOGO1" (at 160.02 172.085 0)
+      (effects (font (size 1.27 1.27)) (justify left))
+    )
+    (property "Value" "~" (at 158.75 175.26 0)
+      (effects (font (size 1.27 1.27)))
+    )
+    (property "Footprint" "logo:logo_15x9" (at 158.75 175.26 0)
+      (effects (font (size 1.27 1.27)) hide)
+    )
+    (property "Datasheet" "" (at 158.75 175.26 0)
+      (effects (font (size 1.27 1.27)) hide)
+    )
+    (instances
+      (project "nrf52840_dev"
+        (path "/e338db97-b3ab-4715-9f06-b1203e9e7bf0"
+          (reference "LOGO1") (unit 1)
+        )
+      )
+    )
+  )
   (symbol (lib_id "Power_Protection:NUP2105L") (at 262.89 55.88 0) (unit 1)
     (in_bom yes) (on_board yes) (dnp no)
@@
   )
   (symbol (lib_id "Mechanical:MountingHole_Pad") (at 130.81 172.72 0) (unit 1)
-    (in_bom yes) (on_board yes) (dnp no) (fields_autoplaced)
+    (in_bom no) (on_board yes) (dnp no) (fields_autoplaced)
     (property "Reference" "H1" (at 133.985 170.18 0)
       (effects (font (size 1.27 1.27)) (justify left))

Commit message: Update production files, add schematic
Signed-off-by: Sergey Terentiev <sergey@terentiev.me>
Other:
- title: (none) -> RC CAN and GPS BLE
Changed lines of the file:
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@@
 (kicad_sch (version 20230121) (generator eeschema)
   (paper "A4")
+  (title_block
+    (title "RC CAN and GPS BLE")
+    (date "2023-07-25")
+  )
   (junction (at 151.765 67.945) (diameter 0) (color 0 0 0 0)
   )
