File: s1st14.kicad_sch (KiCad schematic)
At the start: 19 parts, among them Q5 AO3401A, U3 ST1S14PHR_MY, U4 NCP3335

Commit message: fixes
Parts:
- C12: value 4.7uF -> 10uF
- C14, C18, C19: footprint Capacitor_SMD:C_0603_1608Metric -> Capacitor_SMD:C_0805_2012Metric
Changed lines of the file:
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@@
       (effects (font (size 1.27 1.27)))
     )
-    (property "Footprint" "Capacitor_SMD:C_0603_1608Metric" (at 148.59 76.835 0)
+    (property "Footprint" "Capacitor_SMD:C_0805_2012Metric" (at 148.59 76.835 0)
       (effects (font (size 1.27 1.27)) hide)
     )
@@
       (effects (font (size 1.27 1.27)) (justify left))
     )
-    (property "Value" "4.7uF" (at 108.204 99.314 0)
+    (property "Value" "10uF" (at 108.204 99.314 0)
       (effects (font (size 1.27 1.27)) (justify left))
     )
@@
       (effects (font (size 1.27 1.27)) (justify left))
     )
-    (property "Footprint" "Capacitor_SMD:C_0603_1608Metric" (at 148.59 145.415 0)
+    (property "Footprint" "Capacitor_SMD:C_0805_2012Metric" (at 148.59 145.415 0)
       (effects (font (size 1.27 1.27)) hide)
     )
@@
       (effects (font (size 1.27 1.27)) (justify left))
     )
-    (property "Footprint" "Capacitor_SMD:C_0603_1608Metric" (at 71.12 147.32 0)
-      (effects (font (size 1.27 1.27)) hide)
-    )
+    (property "Footprint" "Capacitor_SMD:C_0805_2012Metric" (at 71.12 147.32 0)
+      (effects (font (size 1.27 1.27)) hide)
+    )

Commit message: Update production files, add schematic
Signed-off-by: Sergey Terentiev <sergey@terentiev.me>
Other:
- title: DASH v2 -> RC CAN and GPS BLE
Changed lines of the file:
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@@
   (paper "A4")
   (title_block
-    (title "DASH v2")
-    (date "2022-08-03")
-    (rev "${GIT_VERSION}")
+    (title "RC CAN and GPS BLE")
+    (date "2023-07-25")
+    (comment 1 "DC/DC ")
   )
   (junction (at 98.425 92.075) (diameter 0) (color 0 0 0 0)
