File: ubloxM8N.kicad_sch (KiCad schematic)
At the start: 5 parts, among them U17 NEO-8M

Commit message: fixes
Parts:
- C40: footprint Capacitor_SMD:C_0805_2012Metric -> Capacitor_SMD:C_0603_1608Metric
- C49: footprint Capacitor_SMD:C_0603_1608Metric -> Capacitor_SMD:C_0805_2012Metric
Changed lines of the file:
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@@
       (effects (font (size 1.27 1.27)) (justify left))
     )
-    (property "Footprint" "Capacitor_SMD:C_0805_2012Metric" (at 105.41 90.17 0)
+    (property "Footprint" "Capacitor_SMD:C_0603_1608Metric" (at 105.41 90.17 0)
       (effects (font (size 1.27 1.27)) hide)
     )
@@
       (effects (font (size 1.27 1.27)) (justify left))
     )
-    (property "Footprint" "Capacitor_SMD:C_0603_1608Metric" (at 173.99 73.66 0)
+    (property "Footprint" "Capacitor_SMD:C_0805_2012Metric" (at 173.99 73.66 0)
       (effects (font (size 1.27 1.27)) hide)
     )

Commit message: Update production files, add schematic
Signed-off-by: Sergey Terentiev <sergey@terentiev.me>
Other:
- title: DASH v2 -> RC CAN and GPS BLE
Changed lines of the file:
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@@
   (paper "A4")
   (title_block
-    (title "DASH v2")
-    (date "2022-08-03")
-    (rev "${GIT_VERSION}")
+    (title "RC CAN and GPS BLE")
+    (date "2023-07-25")
+    (comment 1 "Ublox GPS Recevier")
   )
   (junction (at 165.1 101.6) (diameter 0) (color 0 0 0 0)
